File: PCB/kicad_piscinador_v001/kicad_test_picinador.kicad_pcb (KiCad board)
At the start: 2 copper layers, 48.3 x 35.6 mm, 2 parts, among them U1 DG441, U2 DG441

Commit message: bk pcb
Connections:
- U2 pad 8: Net-(U2-Pad8) -> Net-(U2-Pad4)
Routing:
- net Net-(U2-Pad4): track 0.00 -> 10.6 mm, vias 0 -> 2
Changed lines of the file:
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@@
 (kicad_pcb (version 4) (host pcbnew 4.0.4+e1-6308~48~ubuntu14.04.1-stable)
   (general
-    (links 6)
+    (links 7)
     (no_connects 0)
     (area 132.004999 83.744999 180.415001 119.455001)
     (thickness 1.6)
     (drawings 5)
-    (tracks 48)
+    (tracks 57)
     (zones 0)
     (modules 2)
-    (nets 16)
+    (nets 15)
   )
   (page A4)
@@
   (net 8 "Net-(U2-Pad9)")
   (net 9 "Net-(U2-Pad2)")
-  (net 10 "Net-(U2-Pad8)")
-  (net 11 "Net-(U2-Pad15)")
-  (net 12 "Net-(U2-Pad16)")
-  (net 13 "Net-(U2-Pad4)")
-  (net 14 "Net-(U1-Pad13)")
-  (net 15 "Net-(U2-Pad13)")
+  (net 10 "Net-(U2-Pad15)")
+  (net 11 "Net-(U2-Pad16)")
+  (net 12 "Net-(U2-Pad4)")
+  (net 13 "Net-(U1-Pad13)")
+  (net 14 "Net-(U2-Pad13)")
   (net_class Default "This is the default net class."
     (clearance 0.2)
@@
     (add_net "Net-(U2-Pad2)")
     (add_net "Net-(U2-Pad4)")
-    (add_net "Net-(U2-Pad8)")
     (add_net "Net-(U2-Pad9)")
   )
@@
       (net 3 "Net-(U1-Pad3)"))
     (pad 13 smd rect (at -0.635 -2.6 270) (size 0.6 2.2) (layers F.Cu F.Paste F.Mask)
-      (net 14 "Net-(U1-Pad13)"))
+      (net 13 "Net-(U1-Pad13)"))
     (pad 4 smd rect (at -0.635 2.6 270) (size 0.6 2.2) (layers F.Cu F.Paste F.Mask)
       (net 4 "Net-(U1-Pad4)"))
@@
     (fp_line (start 6.745 -0.23) (end -5.745 -0.23) (layer F.SilkS) (width 0.15))
     (pad 16 smd rect (at -4.445 -2.6 90) (size 0.6 2.2) (layers F.Cu F.Paste F.Mask)
-      (net 12 "Net-(U2-Pad16)"))
+      (net 11 "Net-(U2-Pad16)"))
     (pad 1 smd rect (at -4.445 2.6 90) (size 0.6 2.2) (layers F.Cu F.Paste F.Mask)
       (net 7 "Net-(U2-Pad1)"))
     (pad 15 smd rect (at -3.175 -2.6 90) (size 0.6 2.2) (layers F.Cu F.Paste F.Mask)
-      (net 11 "Net-(U2-Pad15)"))
+      (net 10 "Net-(U2-Pad15)"))
     (pad 2 smd rect (at -3.175 2.6 90) (size 0.6 2.2) (layers F.Cu F.Paste F.Mask)
       (net 9 "Net-(U2-Pad2)"))
@@
       (net 6 "Net-(U2-Pad10)"))
     (pad 3 smd rect (at -1.905 2.6 90) (size 0.6 2.2) (layers F.Cu F.Paste F.Mask)
-      (net 11 "Net-(U2-Pad15)"))
+      (net 10 "Net-(U2-Pad15)"))
     (pad 13 smd rect (at -0.635 -2.6 90) (size 0.6 2.2) (layers F.Cu F.Paste F.Mask)
-      (net 15 "Net-(U2-Pad13)"))
+      (net 14 "Net-(U2-Pad13)"))
     (pad 4 smd rect (at -0.635 2.6 90) (size 0.6 2.2) (layers F.Cu F.Paste F.Mask)
-      (net 13 "Net-(U2-Pad4)"))
+      (net 12 "Net-(U2-Pad4)"))
     (pad 12 smd rect (at 0.635 -2.6 90) (size 0.6 2.2) (layers F.Cu F.Paste F.Mask))
     (pad 5 smd rect (at 0.635 2.6 90) (size 0.6 2.2) (layers F.Cu F.Paste F.Mask)
@@
       (net 6 "Net-(U2-Pad10)"))
     (pad 7 smd rect (at 3.175 2.6 90) (size 0.6 2.2) (layers F.Cu F.Paste F.Mask)
-      (net 12 "Net-(U2-Pad16)"))
+      (net 11 "Net-(U2-Pad16)"))
     (pad 9 smd rect (at 4.445 -2.6 90) (size 0.6 2.2) (layers F.Cu F.Paste F.Mask)
       (net 8 "Net-(U2-Pad9)"))
     (pad 8 smd rect (at 4.445 2.6 90) (size 0.6 2.2) (layers F.Cu F.Paste F.Mask)
-      (net 10 "Net-(U2-Pad8)"))
+      (net 12 "Net-(U2-Pad4)"))
   )
   (gr_line (start 132.08 86.36) (end 132.08 83.82) (angle 90) (layer Edge.Cuts) (width 0.15))
@@
   (via (at 153.67 100.33) (size 0.6) (drill 0.4) (layers F.Cu B.Cu) (net 5))
   (segment (start 153.035 99.695) (end 153.67 100.33) (width 0.25) (layer F.Cu) (net 5))
-  (segment (start 144.72 97.155) (end 146.685 97.155) (width 0.25) (layer F.Cu) (net 6) (status 400000))
+  (segment (start 144.72 97.155) (end 146.685 97.155) (width 0.25) (layer F.Cu) (net 6))
   (segment (start 146.685 97.155) (end 147.955 98.425) (width 0.25) (layer F.Cu) (net 6))
-  (segment (start 147.955 98.425) (end 149.92 98.425) (width 0.25) (layer F.Cu) (net 6) (status 800000))
+  (segment (start 147.955 98.425) (end 149.92 98.425) (width 0.25) (layer F.Cu) (net 6))
   (segment (start 144.72 102.235) (end 146.685 102.235) (width 0.25) (layer F.Cu) (net 6))
   (segment (start 147.955 98.425) (end 149.92 98.425) (width 0.25) (layer F.Cu) (net 6))
@@
   (segment (start 147.32 101.6) (end 147.32 99.06) (width 0.25) (layer F.Cu) (net 6))
   (segment (start 146.685 102.235) (end 147.32 101.6) (width 0.25) (layer F.Cu) (net 6))
-  (segment (start 149.92 102.235) (end 151.765 102.235) (width 0.25) (layer F.Cu) (net 11))
-  (segment (start 142.875 103.505) (end 144.72 103.505) (width 0.25) (layer F.Cu) (net 11))
-  (segment (start 142.24 104.14) (end 142.875 103.505) (width 0.25) (layer F.Cu) (net 11))
-  (via (at 142.24 104.14) (size 0.6) (drill 0.4) (layers F.Cu B.Cu) (net 11))
-  (segment (start 142.24 107.95) (end 142.24 104.14) (width 0.25) (layer B.Cu) (net 11))
-  (segment (start 143.51 109.22) (end 142.24 107.95) (width 0.25) (layer B.Cu) (net 11))
-  (segment (start 152.4 109.22) (end 143.51 109.22) (width 0.25) (layer B.Cu) (net 11))
-  (segment (start 152.4 106.68) (end 152.4 109.22) (width 0.25) (layer B.Cu) (net 11))
-  (via (at 152.4 106.68) (size 0.6) (drill 0.4) (layers F.Cu B.Cu) (net 11))
-  (segment (start 152.4 102.87) (end 152.4 106.68) (width 0.25) (layer F.Cu) (net 11))
-  (segment (start 151.765 102.235) (end 152.4 102.87) (width 0.25) (layer F.Cu) (net 11))
-  (segment (start 149.92 97.155) (end 154.305 97.155) (width 0.25) (layer F.Cu) (net 12))
-  (segment (start 144.72 106.62) (end 144.72 104.775) (width 0.25) (layer F.Cu) (net 12))
-  (segment (start 146.05 107.95) (end 144.72 106.62) (width 0.25) (layer F.Cu) (net 12))
-  (segment (start 153.67 107.95) (end 146.05 107.95) (width 0.25) (layer F.Cu) (net 12))
-  (segment (start 154.94 106.68) (end 153.67 107.95) (width 0.25) (layer F.Cu) (net 12))
-  (segment (start 154.94 97.79) (end 154.94 106.68) (width 0.25) (layer F.Cu) (net 12))
-  (segment (start 154.305 97.155) (end 154.94 97.79) (width 0.25) (layer F.Cu) (net 12))
+  (segment (start 149.92 102.235) (end 151.765 102.235) (width 0.25) (layer F.Cu) (net 10))
+  (segment (start 142.875 103.505) (end 144.72 103.505) (width 0.25) (layer F.Cu) (net 10))
+  (segment (start 142.24 104.14) (end 142.875 103.505) (width 0.25) (layer F.Cu) (net 10))
+  (via (at 142.24 104.14) (size 0.6) (drill 0.4) (layers F.Cu B.Cu) (net 10))
+  (segment (start 142.24 107.95) (end 142.24 104.14) (width 0.25) (layer B.Cu) (net 10))
+  (segment (start 143.51 109.22) (end 142.24 107.95) (width 0.25) (layer B.Cu) (net 10))
+  (segment (start 152.4 109.22) (end 143.51 109.22) (width 0.25) (layer B.Cu) (net 10))
+  (segment (start 152.4 106.68) (end 152.4 109.22) (width 0.25) (layer B.Cu) (net 10))
+  (via (at 152.4 106.68) (size 0.6) (drill 0.4) (layers F.Cu B.Cu) (net 10))
+  (segment (start 152.4 102.87) (end 152.4 106.68) (width 0.25) (layer F.Cu) (net 10))
+  (segment (start 151.765 102.235) (end 152.4 102.87) (width 0.25) (layer F.Cu) (net 10))
+  (segment (start 149.92 97.155) (end 154.305 97.155) (width 0.25) (layer F.Cu) (net 11))
+  (segment (start 144.72 106.62) (end 144.72 104.775) (width 0.25) (layer F.Cu) (net 11))
+  (segment (start 146.05 107.95) (end 144.72 106.62) (width 0.25) (layer F.Cu) (net 11))
+  (segment (start 153.67 107.95) (end 146.05 107.95) (width 0.25) (layer F.Cu) (net 11))
+  (segment (start 154.94 106.68) (end 153.67 107.95) (width 0.25) (layer F.Cu) (net 11))
+  (segment (start 154.94 97.79) (end 154.94 106.68) (width 0.25) (layer F.Cu) (net 11))
+  (segment (start 154.305 97.155) (end 154.94 97.79) (width 0.25) (layer F.Cu) (net 11))
+  (segment (start 149.92 95.885) (end 151.765 95.885) (width 0.25) (layer F.Cu) (net 12) (status 400000))
+  (segment (start 151.765 100.965) (end 149.92 100.965) (width 0.25) (layer F.Cu) (net 12) (status 800000))
+  (segment (start 152.4 101.6) (end 151.765 100.965) (width 0.25) (layer F.Cu) (net 12))
+  (segment (start 152.4 100.33) (end 152.4 101.6) (width 0.25) (layer F.Cu) (net 12))
+  (via (at 152.4 100.33) (size 0.6) (drill 0.4) (layers F.Cu B.Cu) (net 12))
+  (segment (start 152.4 97.79) (end 152.4 100.33) (width 0.25) (layer B.Cu) (net 12))
+  (segment (start 152.4 96.52) (end 152.4 97.79) (width 0.25) (layer B.Cu) (net 12))
+  (via (at 152.4 96.52) (size 0.6) (drill 0.4) (layers F.Cu B.Cu) (net 12))
+  (segment (start 151.765 95.885) (end 152.4 96.52) (width 0.25) (layer F.Cu) (net 12))
 )

Commit message: pcb project
Connections:
- U2 pad 8: Net-(U2-Pad4) -> Net-(U2-Pad8)
Routing:
- net Net-(U2-Pad4): track 10.6 -> 0.00 mm, vias 2 -> 0
Changed lines of the file:
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@@
 (kicad_pcb (version 4) (host pcbnew 4.0.4+e1-6308~48~ubuntu14.04.1-stable)
   (general
-    (links 7)
+    (links 6)
     (no_connects 0)
     (area 132.004999 83.744999 180.415001 119.455001)
     (thickness 1.6)
     (drawings 5)
-    (tracks 57)
+    (tracks 48)
     (zones 0)
     (modules 2)
-    (nets 15)
+    (nets 16)
   )
   (page A4)
@@
   (net 13 "Net-(U1-Pad13)")
   (net 14 "Net-(U2-Pad13)")
+  (net 15 "Net-(U2-Pad8)")
   (net_class Default "This is the default net class."
     (clearance 0.2)
@@
     (add_net "Net-(U2-Pad2)")
     (add_net "Net-(U2-Pad4)")
+    (add_net "Net-(U2-Pad8)")
     (add_net "Net-(U2-Pad9)")
   )
@@
       (net 8 "Net-(U2-Pad9)"))
     (pad 8 smd rect (at 4.445 2.6 90) (size 0.6 2.2) (layers F.Cu F.Paste F.Mask)
-      (net 12 "Net-(U2-Pad4)"))
+      (net 15 "Net-(U2-Pad8)"))
   )
   (gr_line (start 132.08 86.36) (end 132.08 83.82) (angle 90) (layer Edge.Cuts) (width 0.15))
@@
   (segment (start 154.94 97.79) (end 154.94 106.68) (width 0.25) (layer F.Cu) (net 11))
   (segment (start 154.305 97.155) (end 154.94 97.79) (width 0.25) (layer F.Cu) (net 11))
-  (segment (start 149.92 95.885) (end 151.765 95.885) (width 0.25) (layer F.Cu) (net 12) (status 400000))
-  (segment (start 151.765 100.965) (end 149.92 100.965) (width 0.25) (layer F.Cu) (net 12) (status 800000))
-  (segment (start 152.4 101.6) (end 151.765 100.965) (width 0.25) (layer F.Cu) (net 12))
-  (segment (start 152.4 100.33) (end 152.4 101.6) (width 0.25) (layer F.Cu) (net 12))
-  (via (at 152.4 100.33) (size 0.6) (drill 0.4) (layers F.Cu B.Cu) (net 12))
-  (segment (start 152.4 97.79) (end 152.4 100.33) (width 0.25) (layer B.Cu) (net 12))
-  (segment (start 152.4 96.52) (end 152.4 97.79) (width 0.25) (layer B.Cu) (net 12))
-  (via (at 152.4 96.52) (size 0.6) (drill 0.4) (layers F.Cu B.Cu) (net 12))
-  (segment (start 151.765 95.885) (end 152.4 96.52) (width 0.25) (layer F.Cu) (net 12))
 )
