File: PCB/kicad_piscinador_v001/BatteryCharger.sch (KiCad schematic (older format))
At the start: 9 parts

Commit message: try
Connections:
- wire segments 30 -> 36
Other:
- note added: "it shall work with 3.3 or 4.5 battery packs"
- moved on the sheet: BAT?, R?, U?
Changed lines of the file:
@@
 L BATTERY BAT?
 U 1 1 57FFC7C9
-P 6350 3150
-F 0 "BAT?" H 6350 3350 50  0000 C CNN
-F 1 "BATTERY" H 6350 2960 50  0000 C CNN
-F 2 "" H 6350 3150 60  0000 C CNN
-F 3 "" H 6350 3150 60  0000 C CNN
-F 4 "Samsumg" H 6350 3150 60  0001 C CNN "Manufacturer"
-	1    6350 3150
+P 8350 3150
+F 0 "BAT?" H 8350 3350 50  0000 C CNN
+F 1 "BATTERY" H 8350 2960 50  0000 C CNN
+F 2 "" H 8350 3150 60  0000 C CNN
+F 3 "" H 8350 3150 60  0000 C CNN
+F 4 "Samsumg" H 8350 3150 60  0001 C CNN "Manufacturer"
+	1    8350 3150
 	0    1    1    0
 $EndComp
@@
 L LTC3121 U?
 U 1 1 58028389
-P 8000 3100
-F 0 "U?" H 8050 3700 60  0000 C CNN
-F 1 "LTC3121" H 7950 3400 60  0000 C CNN
-F 2 "12-Lead (4mm × 3mm) Plastic DFN" H 8000 3100 60  0001 C CNN
-F 3 "" H 8000 3100 60  0001 C CNN
-F 4 "Linear" H 8000 3100 60  0001 C CNN "Manufaturer"
-F 5 "LTC3121EDE#PBF" H 8000 3100 60  0001 C CNN "Manufacurer No"
-	1    8000 3100
+P 8850 3100
+F 0 "U?" H 8900 3700 60  0000 C CNN
+F 1 "LTC3121" H 8800 3400 60  0000 C CNN
+F 2 "12-Lead (4mm × 3mm) Plastic DFN" H 8850 3100 60  0001 C CNN
+F 3 "" H 8850 3100 60  0001 C CNN
+F 4 "Linear" H 8850 3100 60  0001 C CNN "Manufaturer"
+F 5 "LTC3121EDE#PBF" H 8850 3100 60  0001 C CNN "Manufacurer No"
+	1    8850 3100
 	1    0    0    -1
 $EndComp
@@
 L CRCW0603150RFKEA R?
 U 1 1 58028919
-P 8850 3750
-F 0 "R?" H 8700 3829 50  0000 L CNN
-F 1 "CRCW0603150RFKEA" H 8550 3600 50  0000 L CNN
-F 2 "CRCW0603150RFKEA_RESC1608X55" H 8850 3750 50  0001 L CNN
-F 3 "VISHAY" H 8850 3750 50  0001 L CNN
-	1    8850 3750
+P 9700 3750
+F 0 "R?" H 9550 3829 50  0000 L CNN
+F 1 "CRCW0603150RFKEA" H 9400 3600 50  0000 L CNN
+F 2 "CRCW0603150RFKEA_RESC1608X55" H 9700 3750 50  0001 L CNN
+F 3 "VISHAY" H 9700 3750 50  0001 L CNN
+	1    9700 3750
 	0    1    1    0
 $EndComp
@@
 L CRCW0603150RFKEA R?
 U 1 1 58028B0E
-P 9350 3750
-F 0 "R?" H 9200 3829 50  0000 L CNN
-F 1 "CRCW0603150RFKEA" H 9000 3600 50  0000 L CNN
-F 2 "CRCW0603150RFKEA_RESC1608X55" H 9350 3750 50  0001 L CNN
-F 3 "VISHAY" H 9350 3750 50  0001 L CNN
-	1    9350 3750
+P 10200 3750
+F 0 "R?" H 10050 3829 50  0000 L CNN
+F 1 "CRCW0603150RFKEA" H 9850 3600 50  0000 L CNN
+F 2 "CRCW0603150RFKEA_RESC1608X55" H 10200 3750 50  0001 L CNN
+F 3 "VISHAY" H 10200 3750 50  0001 L CNN
+	1    10200 3750
 	0    1    1    0
 $EndComp
 Wire Wire Line
-	7200 3300 7200 3650
+	8050 3300 8050 3650
 Wire Wire Line
-	7200 3300 7500 3300
+	8050 3300 8350 3300
 Wire Wire Line
-	7900 3600 7900 4650
+	8750 4650 8750 3600
 Wire Wire Line
-	5600 4650 6350 4650
+	7600 4650 8050 4650
 Wire Wire Line
-	6350 4650 7200 4650
+	8050 4650 8350 4650
 Wire Wire Line
-	7200 4650 7900 4650
+	8350 4650 8050 4650
 Wire Wire Line
-	7900 4650 8000 4650
+	8050 4650 8350 4650
 Wire Wire Line
-	8000 4650 8100 4650
+	8350 4650 8750 4650
 Wire Wire Line
-	8100 4650 8850 4650
+	8750 4650 8850 4650
 Wire Wire Line
-	8850 4650 9350 4650
+	8850 4650 8950 4650
 Wire Wire Line
-	9350 4650 10750 4650
+	8950 4650 9700 4650
 Wire Wire Line
-	8000 3600 8000 4650
+	9700 4650 10200 4650
 Wire Wire Line
-	8100 3600 8100 4650
-Connection ~ 8000 4650
-Connection ~ 7900 4650
+	10200 4650 10750 4650
 Wire Wire Line
-	8550 3300 8850 3300
+	8850 3600 8850 4650
 Wire Wire Line
-	8850 3300 8850 3450
-Connection ~ 8100 4650
+	8950 3600 8950 4650
+Connection ~ 8850 4650
+Connection ~ 8750 4650
 Wire Wire Line
-	8550 2700 8550 2550
+	9400 3300 9700 3300
 Wire Wire Line
-	9350 2550 10500 2550
+	9700 3300 9700 3450
+Connection ~ 8950 4650
 Wire Wire Line
-	8550 3050 9000 3050
+	9400 2700 9400 2550
 Wire Wire Line
-	8550 3200 9350 3200
+	9400 2550 9600 2550
 Wire Wire Line
-	9350 3200 9350 3450
-$Comp
-L C C?
-U 1 1 5803755E
-P 8750 2800
-F 0 "C?" H 8775 2900 50  0000 L CNN
-F 1 "C" H 8775 2700 50  0000 L CNN
-F 2 "" H 8788 2650 50  0000 C CNN
-F 3 "" H 8750 2800 50  0000 C CNN
-	1    8750 2800
-	1    0    0    -1
-$EndComp
+	9600 2550 10200 2550
+Wire Wire Line
+	10200 2550 10500 2550
+Wire Wire Line
+	9400 3200 10200 3200
+Wire Wire Line
+	10200 3200 10200 3450
 $Comp
 L C C?
 U 1 1 5803780A
-P 8850 4300
-F 0 "C?" H 8875 4400 50  0000 L CNN
-F 1 "C" H 8875 4200 50  0000 L CNN
-F 2 "" H 8888 4150 50  0000 C CNN
-F 3 "" H 8850 4300 50  0000 C CNN
-	1    8850 4300
+P 9700 4300
+F 0 "C?" H 9725 4400 50  0000 L CNN
+F 1 "C" H 9725 4200 50  0000 L CNN
+F 2 "" H 9738 4150 50  0000 C CNN
+F 3 "" H 9700 4300 50  0000 C CNN
+	1    9700 4300
 	1    0    0    -1
 $EndComp
@@
 L C C?
 U 1 1 58037850
-P 7200 3800
-F 0 "C?" H 7225 3900 50  0000 L CNN
-F 1 "C" H 7225 3700 50  0000 L CNN
-F 2 "" H 7238 3650 50  0000 C CNN
-F 3 "" H 7200 3800 50  0000 C CNN
-	1    7200 3800
+P 8050 3800
+F 0 "C?" H 8075 3900 50  0000 L CNN
+F 1 "C" H 8075 3700 50  0000 L CNN
+F 2 "" H 8088 3650 50  0000 C CNN
+F 3 "" H 8050 3800 50  0000 C CNN
+	1    8050 3800
 	1    0    0    -1
 $EndComp
 Wire Wire Line
-	8850 4050 8850 4150
+	9700 4050 9700 4150
 Wire Wire Line
-	9350 4050 9350 4650
-Connection ~ 9350 4650
+	10200 4050 10200 4650
+Connection ~ 10200 4650
 Wire Wire Line
-	8850 4450 8850 4650
-Connection ~ 8850 4650
+	9700 4450 9700 4650
+Connection ~ 9700 4650
 Wire Wire Line
-	7200 3950 7200 4650
+	8050 3950 8050 4650
 $Comp
 L CRCW0603150RFKEA R?
 U 1 1 58037C47
-P 9350 2900
-F 0 "R?" H 9200 2979 50  0000 L CNN
-F 1 "CRCW0603150RFKEA" H 9000 2750 50  0000 L CNN
-F 2 "CRCW0603150RFKEA_RESC1608X55" H 9350 2900 50  0001 L CNN
-F 3 "VISHAY" H 9350 2900 50  0001 L CNN
-	1    9350 2900
+P 10200 2900
+F 0 "R?" H 10050 2979 50  0000 L CNN
+F 1 "CRCW0603150RFKEA" H 9850 2750 50  0000 L CNN
+F 2 "CRCW0603150RFKEA_RESC1608X55" H 10200 2900 50  0001 L CNN
+F 3 "VISHAY" H 10200 2900 50  0001 L CNN
+	1    10200 2900
 	0    1    1    0
 $EndComp
 Wire Wire Line
-	9350 2600 9350 2550
+	10200 2600 10200 2550
 Wire Notes Line
 	6950 5150 6950 5150
@@
 L CON_JACK_MONO_SW P?
 U 1 1 58037EB1
-P 5100 2800
-F 0 "P?" H 4750 3050 60  0000 C CNN
-F 1 "CON_JACK_MONO_SW" H 5150 2600 60  0000 C CNN
-F 2 "" H 5100 2800 60  0000 C CNN
-F 3 "" H 5100 2800 60  0000 C CNN
-	1    5100 2800
+P 7100 2800
+F 0 "P?" H 6750 3050 60  0000 C CNN
+F 1 "CON_JACK_MONO_SW" H 7150 2600 60  0000 C CNN
+F 2 "" H 7100 2800 60  0000 C CNN
+F 3 "" H 7100 2800 60  0000 C CNN
+	1    7100 2800
 	1    0    0    1
 $EndComp
 Wire Wire Line
-	5600 2700 7350 2700
-Connection ~ 7200 4650
+	7600 2700 8200 2700
+Connection ~ 8050 4650
 Wire Wire Line
-	5600 2950 5600 4650
-Connection ~ 6350 4650
+	7600 2950 7600 4650
+Connection ~ 8350 4650
 Wire Wire Line
-	5600 2800 6350 2800
+	7600 2800 8350 2800
 Wire Wire Line
-	6350 2800 6350 2850
+	8350 2800 8350 2850
 Wire Wire Line
-	6350 3450 6350 4650
+	8350 3450 8350 4650
 Text Notes 1200 1000 0    118  ~ 24
 Energy harvesting and battery charger
+Connection ~ 10200 2550
+Wire Wire Line
+	9600 2650 9600 2550
+Connection ~ 9600 2550
+Wire Wire Line
+	9600 2950 9600 3050
+$Comp
+L C C?
+U 1 1 5803755E
+P 9600 2800
+F 0 "C?" H 9625 2900 50  0000 L CNN
+F 1 "C" H 9625 2700 50  0000 L CNN
+F 2 "" H 9638 2650 50  0000 C CNN
+F 3 "" H 9600 2800 50  0000 C CNN
+	1    9600 2800
+	1    0    0    -1
+$EndComp
+Wire Wire Line
+	9600 3050 9400 3050
+Text Notes 5550 5150 0    60   ~ 0
+it shall work with 3.3 or 4.5 battery packs
 $EndSCHEMATC
